File: MainBoard/RADAR_Main_Board/RADAR_Main_Board_3.kicad_sch (KiCad schematic)
At the start: 400 parts, among them J20 142-0731-211, J21 CJT-T-P-HH-ST-TH1, J22 142-0731-211, J23 142-0731-211, J24 142-0731-211, J25 142-0731-211, J26 142-0731-211, J27 142-0731-211, J28 142-0731-211, J29 142-0731-211, J30 142-0731-211, J31 142-0731-211, J32 142-0731-211, J33 142-0731-211, J34 142-0731-211, J35 142-0731-211, J36 142-0731-211, J37 142-0731-211, J38 142-0731-211, J39 142-0731-211, J40 142-0731-211, J41 142-0731-211, J42 142-0731-211, J43 142-0731-211, J44 142-0731-211, J45 142-0731-211, J46 142-0731-211, J47 142-0731-211, J48 142-0731-211, J49 142-0731-211, J50 142-0731-211, J51 142-0731-211, J52 142-0731-211, J53 142-0731-211, J54 142-0731-211, J55 142-0731-211, U1 AD9484BCPZ-500, U13 LTC5552IUDBTRMPBF, U14 SZMMSZ5232BT1G, U15 SZMMSZ5232BT1G, U16 EP4RKU+, U17 SZMMSZ5232BT1G, U3 AD9708AR, U37 SZMMSZ5232BT1G, U38 SZMMSZ5232BT1G, U39 SZMMSZ5232BT1G, U4 AD8352ACPZ-R7, U40 SZMMSZ5232BT1G, U41 SZMMSZ5232BT1G, U43 SZMMSZ5232BT1G, U44 SZMMSZ5232BT1G, U45 SZMMSZ5232BT1G, U46 SZMMSZ5232BT1G, U47 SZMMSZ5232BT1G, U48 SZMMSZ5232BT1G, U49 SZMMSZ5232BT1G, U5 LTC5552IUDBTRMPBF, U50 SZMMSZ5232BT1G, U51 SZMMSZ5232BT1G, U52 SZMMSZ5232BT1G, U53 SZMMSZ5232BT1G, U54 SZMMSZ5232BT1G, U55 SZMMSZ5232BT1G, U56 SZMMSZ5232BT1G, U57 SZMMSZ5232BT1G, U58 SZMMSZ5232BT1G, U59 SZMMSZ5232BT1G, U60 SZMMSZ5232BT1G, U61 SZMMSZ5232BT1G, U62 SZMMSZ5232BT1G, U63 SZMMSZ5232BT1G, U64 SZMMSZ5232BT1G, U65 SZMMSZ5232BT1G, U66 SZMMSZ5232BT1G, U67 SZMMSZ5232BT1G, U68 SZMMSZ5232BT1G, U8 AD8352ACPZ-R7

Commit message: 🤖 AUTOMATED: MainBoard connector addition complete
Fully automated workflow completed:
✅ Connectors added (J_PWR_IN, J_TILE_SYNC, J_PA_BIAS)
✅ Nets connected automatically
✅ PCB updated from schematic
✅ DRC passed
✅ Gerbers exported

No manual work required - all steps automated via Python scripts.

Generated by: auto_workflow.sh
Parts:
- added J_PA_BIAS: Conn_02x10_Odd_Even, Connector_PinHeader_2.54mm:PinHeader_2x10_P2.54mm_Vertical
- added J_TILE_SYNC: Conn_02x25_Odd_Even, Connector_PinHeader_2.54mm:PinHeader_2x25_P2.54mm_Vertical

Commit message: Revert "🤖 AUTOMATED: MainBoard connector addition complete"
This reverts commit 02bcae12662c453d425235cc63a022ba9474ca3a.
Parts:
- removed J_PA_BIAS: Conn_02x10_Odd_Even, Connector_PinHeader_2.54mm:PinHeader_2x10_P2.54mm_Vertical
- removed J_TILE_SYNC: Conn_02x25_Odd_Even, Connector_PinHeader_2.54mm:PinHeader_2x25_P2.54mm_Vertical
