File: Fractal_32x16/BACKPLANE_16T_v1.kicad_pcb (KiCad board)
At the start: 2 copper layers, 300 x 360 mm, 0 parts

Commit message: ✅ Add ready boards: BACKPLANE_16T, PowerAmplifier, FreqSynthesizer
- BACKPLANE_16T_v1.kicad_pcb: Motherboard for 16 tiles sync
- PowerAmplifierBoard/RF_PA.kicad_pcb: 10W GaN PA board
- FreqSynthesizer MCP_ROUTED: Clock distribution board
- READY_BOARDS.md: Documentation for ready boards

Status: Ready for production
Date: 2026-04-02

Co-authored-by: Qwen-Coder <qwen-coder@alibabacloud.com>
Other:
- board size 300 x 360 mm -> 300 x 402 mm
